File: LVDS-PMOD.kicad_pcb (KiCad board)
At the start: 2 copper layers, 26 parts, among them J1 302-S341, J2 302-S341, U1 SN65LVDS348, U2 SN65LVDS348, U3 SN65LVDS348, U4 SN65LVDS348, U5 SN65LVDS348, U6 SN65LVDS348, U7 SN65LVDS348, U8 SN65LVDS348

Commit message: v1
Parts:
- R1, R2, R3, R4: moved to B.Cu
- moved U4 84.9 mm to (53.3, 75.3)
- moved R1 77.3 mm to (38.1, 85.1), turned to -90 degrees
- moved U3 75.5 mm to (53.3, 64.8)
- moved U8 74.8 mm to (53.3, 127.3)
- moved R2 74.2 mm to (40.6, 85.1), turned to -90 degrees
- moved R3 73.3 mm to (38.1, 137.1), turned to -90 degrees
- moved PMOD3 70.0 mm to (69.5, 98.4), turned to 180 degrees
- moved R4 69.3 mm to (40.6, 137.1), turned to -90 degrees
- moved U2 67.5 mm to (53.3, 54.3)
- moved J1 66.7 mm to (38.1, 40.6)
- moved U7 61.5 mm to (53.3, 116.8)
- moved U1 61.5 mm to (53.3, 43.8)
- moved PMOD4 57.5 mm to (69.5, 121.3), turned to 180 degrees
- moved C1 56.8 mm to (58.5, 43.8), turned to -90 degrees
- moved C2 53.7 mm to (58.3, 54.3), turned to -90 degrees
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- renumbered PMOD2 to PMOD1, PMOD1 to PMOD2, PMOD4 to PMOD3, PMOD3 to PMOD4
Connections:
- PMOD1 pad 1: /LVDS Port AB/IN1 -> /LVDS Port AB/IN7
- PMOD1 pad 10: /LVDS Port AB/IN8 -> /LVDS Port AB/IN2
- PMOD1 pad 2: /LVDS Port AB/IN3 -> /LVDS Port AB/IN5
- PMOD1 pad 3: /LVDS Port AB/IN5 -> /LVDS Port AB/IN3
- PMOD1 pad 4: /LVDS Port AB/IN7 -> /LVDS Port AB/IN1
- PMOD1 pad 7: /LVDS Port AB/IN2 -> /LVDS Port AB/IN8
- PMOD1 pad 8: /LVDS Port AB/IN4 -> /LVDS Port AB/IN6
- PMOD1 pad 9: /LVDS Port AB/IN6 -> /LVDS Port AB/IN4
- PMOD2 pad 1: /LVDS Port AB/IN9 -> /LVDS Port AB/IN15
- PMOD2 pad 10: /LVDS Port AB/IN16 -> /LVDS Port AB/IN10
- PMOD2 pad 2: /LVDS Port AB/IN11 -> /LVDS Port AB/IN13
- PMOD2 pad 3: /LVDS Port AB/IN13 -> /LVDS Port AB/IN11
- PMOD2 pad 4: /LVDS Port AB/IN15 -> /LVDS Port AB/IN9
- PMOD2 pad 7: /LVDS Port AB/IN10 -> /LVDS Port AB/IN16
- PMOD2 pad 8: /LVDS Port AB/IN12 -> /LVDS Port AB/IN14
- PMOD2 pad 9: /LVDS Port AB/IN14 -> /LVDS Port AB/IN12
- PMOD3 pad 1: /LVDS Port CD/IN1 -> /LVDS Port CD/IN7
- PMOD3 pad 10: /LVDS Port CD/IN8 -> /LVDS Port CD/IN2
- PMOD3 pad 2: /LVDS Port CD/IN3 -> /LVDS Port CD/IN5
- PMOD3 pad 3: /LVDS Port CD/IN5 -> /LVDS Port CD/IN3
- PMOD3 pad 4: /LVDS Port CD/IN7 -> /LVDS Port CD/IN1
- PMOD3 pad 7: /LVDS Port CD/IN2 -> /LVDS Port CD/IN8
- PMOD3 pad 8: /LVDS Port CD/IN4 -> /LVDS Port CD/IN6
- PMOD3 pad 9: /LVDS Port CD/IN6 -> /LVDS Port CD/IN4
- PMOD4 pad 1: /LVDS Port CD/IN9 -> /LVDS Port CD/IN15
- PMOD4 pad 10: /LVDS Port CD/IN16 -> /LVDS Port CD/IN10
- PMOD4 pad 2: /LVDS Port CD/IN11 -> /LVDS Port CD/IN13
- PMOD4 pad 3: /LVDS Port CD/IN13 -> /LVDS Port CD/IN11
- PMOD4 pad 4: /LVDS Port CD/IN15 -> /LVDS Port CD/IN9
- PMOD4 pad 7: /LVDS Port CD/IN10 -> /LVDS Port CD/IN16
- PMOD4 pad 8: /LVDS Port CD/IN12 -> /LVDS Port CD/IN14
- PMOD4 pad 9: /LVDS Port CD/IN14 -> /LVDS Port CD/IN12
Routing:
- net GND: track 0.00 -> 35.9 mm, vias 0 -> 16
- net /LVDS Port AB/IN10: track 0.00 -> 23.7 mm
- net /LVDS Port AB/IN2: track 0.00 -> 21.2 mm
- net /LVDS Port AB/IN9: track 0.00 -> 20.5 mm
- net /LVDS Port AB/IN12: track 0.00 -> 19.7 mm
- net /LVDS Port AB/IN14: track 0.00 -> 19.6 mm
- net /LVDS Port AB/IN4: track 0.00 -> 18.9 mm
- net /LVDS Port AB/IN1: track 0.00 -> 18.2 mm
- net /LVDS Port CD/IN10: track 0.00 -> 18.2 mm
- net /LVDS Port AB/IN11: track 0.00 -> 17.9 mm
- net /LVDS Port AB/IN8: track 0.00 -> 17.9 mm
- net /LVDS Port AB/IN6: track 0.00 -> 17.7 mm
- net /LVDS Port AB/IN16: track 0.00 -> 17.4 mm
- net /LVDS Port CD/IN2: track 0.00 -> 17.3 mm
- net /LVDS Port CD/IN12: track 0.00 -> 17.1 mm
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- added copper zone on In2.Cu, net +3V3A
- added copper zone on In2.Cu, net +3V3B
- added copper zone on In2.Cu, net +3V3C
- added copper zone on In2.Cu, net +3V3D
- added copper zone on B.Cu, net GND
- added copper zone on In1.Cu, net GND
Other:
- board outline added: 42.9 x 110.5 mm
- copper layers 2 -> 4
- board text added: "LVDS Quad PMOD v${REVISION} Noah Paladino"
