File: lvds_port.kicad_sch (KiCad schematic)
At the start: 13 parts, among them J1 302-S341, U1 SN65LVDS348, U2 SN65LVDS348, U3 SN65LVDS348, U4 SN65LVDS348

Commit message: v1
Parts:
- renumbered PMOD2 to PMOD1, PMOD1 to PMOD2
Connections:
- net IN1: now also PMOD1.4 (IOA3); no longer PMOD1.1 (IOA0)
- net IN10: now also PMOD2.10 (IOB3); no longer PMOD2.7 (IOB0)
- net IN11: now also PMOD2.3 (IOA2); no longer PMOD2.2 (IOA1)
- net IN12: now also PMOD2.9 (IOB2); no longer PMOD2.8 (IOB1)
- net IN13: now also PMOD2.2 (IOA1); no longer PMOD2.3 (IOA2)
- net IN14: now also PMOD2.8 (IOB1); no longer PMOD2.9 (IOB2)
- net IN15: now also PMOD2.1 (IOA0); no longer PMOD2.4 (IOA3)
- net IN16: now also PMOD2.7 (IOB0); no longer PMOD2.10 (IOB3)
- net IN2: now also PMOD1.10 (IOB3); no longer PMOD1.7 (IOB0)
- net IN3: now also PMOD1.3 (IOA2); no longer PMOD1.2 (IOA1)
- net IN4: now also PMOD1.9 (IOB2); no longer PMOD1.8 (IOB1)
- net IN5: now also PMOD1.2 (IOA1); no longer PMOD1.3 (IOA2)
- net IN6: now also PMOD1.8 (IOB1); no longer PMOD1.9 (IOB2)
- net IN7: now also PMOD1.1 (IOA0); no longer PMOD1.4 (IOA3)
- net IN8: now also PMOD1.7 (IOB0); no longer PMOD1.10 (IOB3)
- net IN9: now also PMOD2.4 (IOA3); no longer PMOD2.1 (IOA0)
Other:
- company: (none) -> MIT
- title: (none) -> LVDS Quad PMOD
- moved on the sheet: C1, C2, C3, C4, J1, PMOD2, R1, R2, U3, U4
